Commit message: Aruco based visual servoing now supported in python.

File: robot_description/free_flying_kinect.xacro (robot description, xacro)
@@ -8,5 +8,5 @@
 <xacro:property name="height1" value="0.2" /> <!-- Link 1 -->
 <xacro:property name="PI" value="3.1415926535897931"/>
-<xacro:property name="x" value="-6"/>
+<xacro:property name="x" value="-2"/>
 <xacro:property name="y" value="0"/>
 <xacro:property name="z" value="0"/>
@@ -15,5 +15,5 @@
 <xacro:property name="y" value="0"/>
 <!-- Import all Gazebo-customization elements, including Gazebo colors -->
-<xacro:include filename="$(find visual_servoing)/robot_description/free_flying_cam.gazebo" />
+<xacro:include filename="$(find visual_servoing)/robot_description/free_flying_kinect.gazebo" />
 <!--link name="world"/-->
 <!--link name="base_footprint"/-->
@@ -79,5 +79,5 @@
     <!-- these values have to be these values otherwise the gazebo camera image
         won't be aligned properly with the frame it is supposedly originating from -->
-    <origin xyz="0 0 0" rpy="${pi/2} 0 ${-pi/2}"/>
+    <origin xyz="0.1 0 0" rpy="${pi/2} 0 ${-pi/2}"/>
     <parent link="camera_link"/>
     <child link="camera_link_optical"/>
